File: KiCad/geiger_entropy.kicad_pcb (KiCad board)
At the start: 2 copper layers, 114.5 x 130.5 mm, 38 parts, among them J1 AudioJack2, J2 Conn_01x04_Socket, J3 Conn_01x10_Pin, J4 Conn_01x10_Pin, J5 Jack-DC, J6 ICSP, SW1 REV, SW2 FWD, SW3 RESET, U1 LM393, U2 ATmega328-P, U3 L7805, Y1 16MHz

Commit message: Add production files and remove legacy gerbers, bom etc
Routing:
- net /D11/MOSI: track 305.8 -> 152.0 mm
- net /A5: track 74.3 -> 65.4 mm
- net /A4: track 81.1 -> 72.8 mm
- net /RESET: track 131.5 -> 133.1 mm
Changed lines of the file:
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@@
+	)
+	(segment
+		(start 94.8575 94)
+		(end 98.96 98.1025)
+		(width 0.2)
+		(layer "B.Cu")
+		(net "/A4")
 	)
 	(segment
@@
 	)
 	(segment
-		(start 54 86)
-		(end 64 76)
-		(width 0.2)
-		(layer "B.Cu")
-		(net "/A4")
-	)
-	(segment
 		(start 98.96 98.1025)
 		(end 98.96 104.8425)
@@
 	)
 	(segment
-		(start 76.8575 76)
-		(end 98.96 98.1025)
+		(start 49.73 86.27)
+		(end 50 86)
+		(width 0.2)
+		(layer "B.Cu")
+		(net "/A4")
+	)
+	(segment
+		(start 49 86.27)
+		(end 49.73 86.27)
+		(width 0.2)
+		(layer "B.Cu")
+		(net "/A4")
+	)
+	(segment
+		(start 62 94)
+		(end 94.8575 94)
+		(width 0.2)
+		(layer "B.Cu")
+		(net "/A4")
+	)
+	(segment
+		(start 54 86)
+		(end 62 94)
 		(width 0.2)
 		(layer "B.Cu")
@@
 	)
 	(segment
-		(start 64 76)
-		(end 76.8575 76)
-		(width 0.2)
-		(layer "B.Cu")
-		(net "/A4")
-	)
-	(segment
-		(start 49 86.27)
-		(end 49.73 86.27)
-		(width 0.2)
-		(layer "B.Cu")
-		(net "/A4")
-	)
-	(segment
-		(start 49.73 86.27)
-		(end 50 86)
-		(width 0.2)
-		(layer "B.Cu")
-		(net "/A4")
+		(start 54.19 88.81)
+		(end 61.38 96)
+		(width 0.2)
+		(layer "B.Cu")
+		(net "/A5")
+	)
+	(segment
+		(start 91.2 103.3225)
+		(end 91.2 110.0625)
+		(width 0.2)
+		(layer "B.Cu")
+		(net "/A5")
+	)
+	(segment
+		(start 94.3175 96)
+		(end 96.42 98.1025)
+		(width 0.2)
+		(layer "B.Cu")
+		(net "/A5")
 	)
 	(segment
@@
 	)
 	(segment
-		(start 76.3175 78)
-		(end 96.42 98.1025)
-		(width 0.2)
-		(layer "B.Cu")
-		(net "/A5")
-	)
-	(segment
-		(start 91.2 103.3225)
-		(end 91.2 110.0625)
-		(width 0.2)
-		(layer "B.Cu")
-		(net "/A5")
-	)
-	(segment
-		(start 54.19 88.81)
-		(end 65 78)
-		(width 0.2)
-		(layer "B.Cu")
-		(net "/A5")
-	)
-	(segment
 		(start 96.42 98.1025)
 		(end 91.2 103.3225)
@@
 	)
 	(segment
-		(start 65 78)
-		(end 76.3175 78)
+		(start 61.38 96)
+		(end 94.3175 96)
 		(width 0.2)
 		(layer "B.Cu")
@@
 	)
 	(segment
-		(start 97.57 98.578846)
-		(end 86.086346 110.0625)
-		(width 0.2)
-		(layer "F.Cu")
-		(net "/RESET")
-	)
-	(segment
 		(start 55.9775 110)
 		(end 53.33 107.3525)
@@
 	)
 	(segment
-		(start 120.585 40.9925)
-		(end 120.585 74.611154)
+		(start 121.975 39.6025)
+		(end 121.975 40.276154)
 		(width 0.2)
 		(layer "F.Cu")
@@
 	)
 	(segment
-		(start 121.975 39.6025)
+		(start 83.58 110.0625)
+		(end 86.086346 110.0625)
+		(width 0.2)
+		(layer "F.Cu")
+		(net "/RESET")
+	)
+	(segment
+		(start 117 78.196154)
+		(end 117 42.951154)
+		(width 0.2)
+		(layer "F.Cu")
+		(net "/RESET")
+	)
+	(segment
+		(start 97.57 97.626154)
+		(end 117 78.196154)
+		(width 0.2)
+		(layer "F.Cu")
+		(net "/RESET")
+	)
+	(segment
+		(start 118.958654 40.9925)
 		(end 120.585 40.9925)
 		(width 0.2)
@@
 	)
 	(segment
-		(start 120.585 74.611154)
-		(end 97.57 97.626154)
+		(start 117 42.951154)
+		(end 118.958654 40.9925)
 		(width 0.2)
 		(layer "F.Cu")
@@
 	)
 	(segment
-		(start 97.57 97.626154)
-		(end 97.57 98.578846)
-		(width 0.2)
-		(layer "F.Cu")
-		(net "/RESET")
-	)
-	(segment
-		(start 86.086346 110.0625)
-		(end 83.58 110.0625)
+		(start 97.57 98.578846)
+		(end 97.57 97.626154)
 		(width 0.2)
 		(layer "F.Cu")
@@
 	)
 	(segment
+		(start 120.585 40.9925)
+		(end 121.975 39.6025)
+		(width 0.2)
+		(layer "F.Cu")
+		(net "/RESET")
+	)
+	(segment
+		(start 86.086346 110.0625)
+		(end 97.57 98.578846)
+		(width 0.2)
+		(layer "F.Cu")
+		(net "/RESET")
+	)
+	(segment
 		(start 83.5175 110)
 		(end 55.9775 110)
@@
 	)
 	(segment
-		(start 64.954532 80.545468)
-		(end 39 106.5)
+		(start 121 85.2425)
+		(end 121 47.175)
 		(width 0.2)
 		(layer "F.Cu")
@@
 	)
 	(segment
-		(start 39 109)
-		(end 41.1625 111.1625)
+		(start 120.825 47)
+		(end 120.825 43.5325)
 		(width 0.2)
 		(layer "F.Cu")
@@
 	)
 	(segment
-		(start 119.435 42.1425)
-		(end 114 47.5775)
+		(start 121 47.175)
+		(end 120.825 47)
 		(width 0.2)
 		(layer "F.Cu")
@@
 	)
 	(segment
-		(start 89.454532 80.545468)
-		(end 64.954532 80.545468)
+		(start 133.86 98.1025)
+		(end 121 85.2425)
 		(width 0.2)
 		(layer "F.Cu")
@@
 	)
 	(segment
-		(start 39 106.5)
-		(end 39 109)
-		(width 0.2)
-		(layer "F.Cu")
-		(net "/D11{slash}MOSI")
-	)
-	(segment
-		(start 114 47.5775)
-		(end 114 56)
-		(width 0.2)
-		(layer "F.Cu")
-		(net "/D11{slash}MOSI")
-	)
-	(segment
-		(start 41.1625 111.1625)
-		(end 86.694766 111.1625)
-		(width 0.2)
-		(layer "F.Cu")
-		(net "/D11{slash}MOSI")
-	)
-	(segment
-		(start 86.694766 111.1625)
-		(end 94.857266 103)
-		(width 0.2)
-		(layer "F.Cu")
-		(net "/D11{slash}MOSI")
-	)
-	(segment
-		(start 128.9625 103)
-		(end 133.86 98.1025)
-		(width 0.2)
-		(layer "F.Cu")
-		(net "/D11{slash}MOSI")
-	)
-	(segment
-		(start 114 56)
-		(end 89.454532 80.545468)
-		(width 0.2)
-		(layer "F.Cu")
-		(net "/D11{slash}MOSI")
-	)
-	(segment
-		(start 94.857266 103)
-		(end 128.9625 103)
+		(start 120.825 43.5325)
+		(end 119.435 42.1425)
 		(width 0.2)
 		(layer "F.Cu")
@@
 	)
 	(segment
+		(start 123.6275 121.5)
+		(end 121.39 119.2625)
+		(width 0.2)
+		(layer "F.Cu")
+		(net "/Geiger_pulse")
+	)
+	(segment
+		(start 130.940397 119.092103)
+		(end 126.08 123.9525)
+		(width 0.2)
+		(layer "F.Cu")
+		(net "/Geiger_pulse")
+	)
+	(segment
+		(start 126.08 123.9525)
+		(end 123.6275 121.5)
+		(width 0.2)
+		(layer "F.Cu")
+		(net "/Geiger_pulse")
+	)
+	(segment
+		(start 133.407898 119.092103)
+		(end 130.940397 119.092103)
+		(width 0.2)
+		(layer "F.Cu")
+		(net "/Geiger_pulse")
+	)
+	(segment
+		(start 126.08 127)
+		(end 126.08 123.9525)
+		(width 0.2)
+		(layer "F.Cu")
+		(net "/Geiger_pulse")
+	)
+	(segment
 		(start 37 43.5)
 		(end 43.5 43.5)
@@
 	)
 	(segment
-		(start 123.6275 121.5)
-		(end 121.39 119.2625)
-		(width 0.2)
-		(layer "F.Cu")
-		(net "/Geiger_pulse")
-	)
-	(segment
-		(start 130.940397 119.092103)
-		(end 126.08 123.9525)
-		(width 0.2)
-		(layer "F.Cu")
-		(net "/Geiger_pulse")
-	)
-	(segment
-		(start 126.08 123.9525)
-		(end 123.6275 121.5)
-		(width 0.2)
-		(layer "F.Cu")
-		(net "/Geiger_pulse")
-	)
-	(segment
-		(start 133.407898 119.092103)
-		(end 130.940397 119.092103)
-		(width 0.2)
-		(layer "F.Cu")
-		(net "/Geiger_pulse")
-	)
-	(segment
-		(start 126.08 127)
-		(end 126.08 123.9525)
-		(width 0.2)
-		(layer "F.Cu")
-		(net "/Geiger_pulse")
-	)
-	(segment

Commit message: Modify PCB
Parts:
- removed ?: LOGO, Entropy32:wave_packet_logo
- removed J3, J4: Conn_01x10_Pin, Connector_PinHeader_2.54mm:PinHeader_1x10_P2.54mm_Vertical
- removed the REF** at (47.0, 128.0)
- added REF**: OSHW-Logo_5.7x6mm_SilkScreen, Symbol:OSHW-Logo_5.7x6mm_SilkScreen, F.Cu at (121.0, 120.0)
- added REF**: KiCad-Logo2_30mm_SilkScreen, Symbol:KiCad-Logo2_30mm_SilkScreen, B.Cu at (95.0, 79.0)
- moved C7 122.6 mm to (151.0, 88.5)
- moved R9 118.9 mm to (154.0, 108.1)
- moved C9 110.9 mm to (151.0, 85.5), turned to 90 degrees
- moved PWR1 107.8 mm to (139.5, 90.0)
- moved J5 106.6 mm to (145.0, 77.0)
- moved L1 104.1 mm to (144.5, 90.0)
- moved U3 96.9 mm to (140.9, 83.0), turned to 0 degrees
- moved R7 80.1 mm to (122.0, 103.9), turned to -90 degrees
- moved J6 76.9 mm to (73.0, 103.9), turned to 0 degrees
- moved C4 50.6 mm to (129.5, 117.0), turned to 0 degrees
- moved R1 50.3 mm to (145.0, 97.9), turned to -90 degrees
- moved C10 47.5 mm to (113.0, 116.0), turned to -90 degrees
- moved R5 42.7 mm to (151.0, 97.9)
- moved R10 42.4 mm to (157.0, 97.9), turned to -90 degrees
- moved J1 40.1 mm to (153.5, 75.8)
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Routing:
- net /D13/SCK: track 204.8 -> 51.0 mm
- net /D11/MOSI: track 152.0 -> 36.5 mm
- net /RESET: track 133.1 -> 31.4 mm
- net /D9: track 93.2 -> 0.00 mm
- net /D12/MISO: track 122.9 -> 36.9 mm
- net +5V: track 283.8 -> 200.3 mm
- net /D10: track 73.1 -> 0.00 mm
- net Net-(J1-PadS): track 73.0 -> 4.07 mm
- net /D4: track 107.9 -> 39.5 mm
- net /D8: track 63.6 -> 0.00 mm
- net /D7: track 60.1 -> 0.00 mm
- net /D5: track 114.0 -> 54.3 mm
- net /D6: track 56.0 -> 0.00 mm
- net /Geiger_pulse: track 19.0 -> 59.5 mm
- net Net-(L1-A): track 3.26 -> 41.2 mm
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Other:
- board size 114.5 x 130.5 mm -> 112 x 63 mm
- board text added: "RST"
- board text removed: "//// 5V LOGIC ////"
- board text removed: "//// CAUTION ////////////////////// OPERATION MAY CREATE PARALLEL UNIVERSES"
- board text removed: "//// DC //// 9-12V ONLY"
- board text removed: "//// WARNING //// GEIGER COUNTER ONLY DO NOT CONNECT AUDIO"
- board text removed: "A0"
- board text removed: "A1"
- board text removed: "A2"
- board text removed: "A3"
- board text removed: "A4"
- board text removed: "A5"
- board text removed: "D0"
- board text removed: "D1"
- board text removed: "D10"
- board text removed: "D11"
- board text removed: "D12"
- board text removed: "D13"
- board text removed: "D2"
- board text removed: "D3"
- board text removed: "D4"
- board text removed: "D5"
- board text removed: "D6"
- board text removed: "D7"
- board text removed: "D8"
- board text removed: "D9"
- board text removed: "The Universe Bifurcator"
- board text removed: "This device complies with the Heisenberg Uncertainty Principle. Operation is subject to the following: (1) this device may not cause harmful interference with causality, (2) this device must accept any interference received, including unexpected entropy."
- board text removed: "^"

Commit message: Update PCB and generate production files
Parts:
- moved J1 2.00 mm to (153.5, 73.8)
- moved J5 2.00 mm to (145.0, 75.0)
Routing:
- net Net-(U3-IN): track 20.0 -> 22.0 mm
- net Net-(J1-PadS): track 4.07 -> 6.07 mm
- net GND: vias 305 -> 308
Changed lines of the file:
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@@
 	(footprint "Connector_BarrelJack:BarrelJack_Horizontal"
 		(layer "F.Cu")
-		(at 145 77 -90)
+		(at 145 75 -90)
 		(descr "DC Barrel Jack")
 		(tags "Power Jack")
@@
 	(footprint "Connector_Audio:Jack_3.5mm_PJ320E_Horizontal"
 		(layer "F.Cu")
-		(at 153.4675 75.75)
+		(at 153.4675 73.75)
 		(descr "Headphones with microphone connector, 3.5mm, 4 pins (http://www.qingpu-electronics.com/en/products/WQP-PJ320E-177.html)")
 		(tags "3.5mm jack mic microphone phones headphones 4pins audio plug")
@@
 	)
 	(via
+		(at 159 77)
+		(size 0.6)
+		(drill 0.3)
+		(layers "F.Cu" "B.Cu")
+		(free yes)
+		(net "GND")
+	)
+	(via
 		(at 75 116)
 		(size 0.6)
@@
 	)
 	(via
+		(at 153 77)
+		(size 0.6)
+		(drill 0.3)
+		(layers "F.Cu" "B.Cu")
+		(free yes)
+		(net "GND")
+	)
+	(via
 		(at 71 112)
 		(size 0.6)
@@
 	)
 	(via
+		(at 155 77)
+		(size 0.6)
+		(drill 0.3)
+		(layers "F.Cu" "B.Cu")
+		(free yes)
+		(net "GND")
+	)
+	(via
 		(at 124 66)
 		(size 0.6)
@@
 	)
 	(segment
-		(start 140.92 81.08)
-		(end 140.92 83)
+		(start 145 78)
+		(end 145 75)
 		(width 0.2)
 		(layer "F.Cu")
@@
 	)
 	(segment
-		(start 145 77)
-		(end 140.92 81.08)
+		(start 140.92 82.08)
+		(end 145 78)
+		(width 0.2)
+		(layer "F.Cu")
+		(net "Net-(U3-IN)")
+	)
+	(segment
+		(start 140.92 83)
+		(end 140.92 82.08)
 		(width 0.2)
 		(layer "F.Cu")
@@
 	)
 	(segment
-		(start 157.9675 79.9525)
-		(end 157 80.92)
+		(start 157 76.2175)
+		(end 157.9675 75.25)
 		(width 0.2)
 		(layer "F.Cu")
@@
 	)
 	(segment
-		(start 157.9675 77.25)
-		(end 157.9675 79.9525)
+		(start 157 80.92)
+		(end 157 76.2175)
 		(width 0.2)
 		(layer "F.Cu")
